File: geiger.sch (EAGLE design)
At the start: 32 parts, among them IC1 AD8666N, X1 MINI-USB_SHIELD4P-85-32004-10X

Commit message: comperator added
Parts:
- added C13: (no value), resistor:C-EU025-025X050
- added IC3: LM358N, linear:LM358N
- added R12: 3,3k, resistor:R-EU_0207/7
- added R13, R14, R16, R17: 1k, resistor:R-EU_0207/7
- added R15: (no value), pot:TRIM_EU-LI10
Connections:
- new net +3V3: C12.1, IC2.OUT, IC3P.V+, R10.1, R16.2, U$1.VCC
- new net N$17: IC3A.-IN, R12.1, R13.2
- new net N$18: R15.E, R16.1
- new net N$19: C13.2, IC3A.+IN, R15.S
- new net N$21: C13.1, IC3A.OUT, R17.2
- new net N$22: IC3B.+IN, R17.1
- net ANALOG_PULSE: now also R12.2
- net GND: now also IC3P.V-, R13.1, R14.1
- net N$16: now also R14.2, R15.A; no longer C12.1, IC2.OUT, R10.1, U$1.VCC
- net PULSE: now also IC3B.-IN, IC3B.OUT
Changed lines of the file:
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@@
 <part name="C12" library="resistor" deviceset="C-EU" device="025-025X050"/>
 <part name="GND15" library="supply1" deviceset="GND" device=""/>
+<part name="IC3" library="linear" deviceset="LM358" device="N"/>
+<part name="+3V1" library="supply1" deviceset="+3V3" device=""/>
+<part name="+3V2" library="supply1" deviceset="+3V3" device=""/>
+<part name="GND16" library="supply1" deviceset="GND" device=""/>
+<part name="R12" library="resistor" deviceset="R-EU_" device="0207/7" value="3,3k"/>
+<part name="R13" library="resistor" deviceset="R-EU_" device="0207/7" value="1k"/>
+<part name="GND17" library="supply1" deviceset="GND" device=""/>
+<part name="R14" library="resistor" deviceset="R-EU_" device="0207/7" value="1k"/>
+<part name="GND18" library="supply1" deviceset="GND" device=""/>
+<part name="R15" library="pot" deviceset="TRIM_EU-" device="LI10"/>
+<part name="R16" library="resistor" deviceset="R-EU_" device="0207/7" value="1k"/>
+<part name="+3V3" library="supply1" deviceset="+3V3" device=""/>
+<part name="C13" library="resistor" deviceset="C-EU" device="025-025X050"/>
+<part name="R17" library="resistor" deviceset="R-EU_" device="0207/7" value="1k"/>
 </parts>
 <sheets>
@@
 <instance part="C12" gate="G$1" x="33.02" y="119.38"/>
 <instance part="GND15" gate="1" x="33.02" y="111.76"/>
+<instance part="IC3" gate="A" x="172.72" y="22.86" rot="MR180"/>
+<instance part="IC3" gate="B" x="205.74" y="20.32"/>
+<instance part="IC3" gate="P" x="205.74" y="20.32"/>
+<instance part="+3V1" gate="G$1" x="33.02" y="127"/>
+<instance part="+3V2" gate="G$1" x="205.74" y="48.26"/>
+<instance part="GND16" gate="1" x="205.74" y="2.54"/>
+<instance part="R12" gate="G$1" x="139.7" y="25.4" rot="R90"/>
+<instance part="R13" gate="G$1" x="139.7" y="10.16" rot="R90"/>
+<instance part="GND17" gate="1" x="139.7" y="2.54"/>
+<instance part="R14" gate="G$1" x="154.94" y="10.16" rot="R90"/>
+<instance part="GND18" gate="1" x="154.94" y="2.54"/>
+<instance part="R15" gate="1" x="154.94" y="20.32"/>
+<instance part="R16" gate="G$1" x="154.94" y="35.56" rot="R90"/>
+<instance part="+3V3" gate="G$1" x="154.94" y="45.72"/>
+<instance part="C13" gate="G$1" x="172.72" y="35.56" rot="R270"/>
+<instance part="R17" gate="G$1" x="190.5" y="22.86" rot="R180"/>
 </instances>
 <busses>
@@
 <pinref part="C12" gate="G$1" pin="2"/>
 <pinref part="GND15" gate="1" pin="GND"/>
+</segment>
+<segment>
+<pinref part="IC3" gate="P" pin="V-"/>
+<pinref part="GND16" gate="1" pin="GND"/>
+<wire x1="205.74" y1="5.08" x2="205.74" y2="12.7" width="0.1524" layer="91"/>
+</segment>
+<segment>
+<pinref part="R13" gate="G$1" pin="1"/>
+<pinref part="GND17" gate="1" pin="GND"/>
+</segment>
+<segment>
+<pinref part="R14" gate="G$1" pin="1"/>
+<pinref part="GND18" gate="1" pin="GND"/>
 </segment>
 </net>
@@
 <pinref part="IC1" gate="B" pin="OUT"/>
 <junction x="111.76" y="45.72"/>
-<wire x1="111.76" y1="30.48" x2="119.38" y2="30.48" width="0.1524" layer="91"/>
 <junction x="111.76" y="30.48"/>
 <label x="114.3" y="30.48" size="1.778" layer="95"/>
+<pinref part="R12" gate="G$1" pin="2"/>
+<wire x1="111.76" y1="30.48" x2="139.7" y2="30.48" width="0.1524" layer="91"/>
 </segment>
 </net>
@@
 <label x="88.9" y="132.08" size="1.778" layer="95"/>
 </segment>
+<segment>
+<pinref part="IC3" gate="B" pin="-IN"/>
+<wire x1="198.12" y1="17.78" x2="195.58" y2="17.78" width="0.1524" layer="91"/>
+<wire x1="195.58" y1="17.78" x2="195.58" y2="10.16" width="0.1524" layer="91"/>
+<wire x1="195.58" y1="10.16" x2="213.36" y2="10.16" width="0.1524" layer="91"/>
+<pinref part="IC3" gate="B" pin="OUT"/>
+<wire x1="213.36" y1="10.16" x2="213.36" y2="20.32" width="0.1524" layer="91"/>
+<wire x1="213.36" y1="20.32" x2="226.06" y2="20.32" width="0.1524" layer="91"/>
+<junction x="213.36" y="20.32"/>
+<label x="215.9" y="20.32" size="1.778" layer="95"/>
+</segment>
 </net>
 <net name="N$10" class="0">
@@
 </segment>
 </net>
-<net name="N$16" class="0">
+<net name="+3V3" class="0">
 <segment>
 <pinref part="IC2" gate="A" pin="OUT"/>
@@
 <wire x1="33.02" y1="121.92" x2="33.02" y2="124.46" width="0.1524" layer="91"/>
 <junction x="33.02" y="124.46"/>
-</segment>
-</net>
+<pinref part="+3V1" gate="G$1" pin="+3V3"/>
+</segment>
+<segment>
+<pinref part="IC3" gate="P" pin="V+"/>
+<pinref part="+3V2" gate="G$1" pin="+3V3"/>
+<wire x1="205.74" y1="45.72" x2="205.74" y2="27.94" width="0.1524" layer="91"/>
+</segment>
+<segment>
+<pinref part="+3V3" gate="G$1" pin="+3V3"/>
+<pinref part="R16" gate="G$1" pin="2"/>
+<wire x1="154.94" y1="43.18" x2="154.94" y2="40.64" width="0.1524" layer="91"/>
+</segment>
+</net>
+<net name="N$17" class="0">
+<segment>
+<pinref part="R12" gate="G$1" pin="1"/>
+<pinref part="R13" gate="G$1" pin="2"/>
+<wire x1="139.7" y1="20.32" x2="139.7" y2="15.24" width="0.1524" layer="91"/>
+<pinref part="IC3" gate="A" pin="-IN"/>
+<wire x1="165.1" y1="25.4" x2="165.1" y2="27.94" width="0.1524" layer="91"/>
+<wire x1="165.1" y1="27.94" x2="147.32" y2="27.94" width="0.1524" layer="91"/>
+<wire x1="147.32" y1="27.94" x2="147.32" y2="20.32" width="0.1524" layer="91"/>
+<wire x1="147.32" y1="20.32" x2="139.7" y2="20.32" width="0.1524" layer="91"/>
+<junction x="139.7" y="20.32"/>
+</segment>
+</net>
+<net name="N$16" class="0">
+<segment>
+<pinref part="R14" gate="G$1" pin="2"/>
+<pinref part="R15" gate="1" pin="A"/>
+</segment>
+</net>
+<net name="N$18" class="0">
+<segment>
+<pinref part="R16" gate="G$1" pin="1"/>
+<pinref part="R15" gate="1" pin="E"/>
+<wire x1="154.94" y1="30.48" x2="154.94" y2="25.4" width="0.1524" layer="91"/>
+</segment>
+</net>
+<net name="N$19" class="0">
+<segment>
+<pinref part="R15" gate="1" pin="S"/>
+<pinref part="IC3" gate="A" pin="+IN"/>
+<wire x1="160.02" y1="20.32" x2="162.56" y2="20.32" width="0.1524" layer="91"/>
+<pinref part="C13" gate="G$1" pin="2"/>
+<wire x1="162.56" y1="20.32" x2="165.1" y2="20.32" width="0.1524" layer="91"/>
+<wire x1="167.64" y1="35.56" x2="162.56" y2="35.56" width="0.1524" layer="91"/>
+<wire x1="162.56" y1="35.56" x2="162.56" y2="20.32" width="0.1524" layer="91"/>
+<junction x="162.56" y="20.32"/>
+</segment>
+</net>
+<net name="N$21" class="0">
+<segment>
+<pinref part="C13" gate="G$1" pin="1"/>
+<wire x1="175.26" y1="35.56" x2="182.88" y2="35.56" width="0.1524" layer="91"/>
+<wire x1="182.88" y1="35.56" x2="182.88" y2="22.86" width="0.1524" layer="91"/>
+<pinref part="IC3" gate="A" pin="OUT"/>
+<wire x1="182.88" y1="22.86" x2="180.34" y2="22.86" width="0.1524" layer="91"/>
+<pinref part="R17" gate="G$1" pin="2"/>
+<wire x1="185.42" y1="22.86" x2="182.88" y2="22.86" width="0.1524" layer="91"/>
+<junction x="182.88" y="22.86"/>
+</segment>
+</net>
+<net name="N$22" class="0">
+<segment>
+<pinref part="R17" gate="G$1" pin="1"/>
+<pinref part="IC3" gate="B" pin="+IN"/>
+<wire x1="195.58" y1="22.86" x2="198.12" y2="22.86" width="0.1524" layer="91"/>
+</segment>
+</net>
